File: schematic_pcb/robohand/robohand.kicad_sch (KiCad schematic)
At the start: 10 parts, among them M1 Motor_Servo, M2 Motor_Servo, M3 Motor_Servo, M4 Motor_Servo, M5 Motor_Servo, SW1 SW_SPST, SW2 SW_SPST, SW3 SW_SPST, U1 ESP32-CAM

Commit message: august 6th - some schematci and BOM editing
Parts:
- removed SW1, SW2, SW3: SW_SPST, Button_Switch_THT:SW_PUSH_6mm_H5mm, symbol Switch:SW_SPST
- added M10, M6, M7, M8, M9: Motor_Servo, Connector_PinHeader_2.54mm:PinHeader_1x03_P2.54mm_Vertical, symbol Motor:Motor_Servo
- added MyoWare EMG Sensor1: ~, symbol MyoWare_EMG_Sensor:MyoWare_EMG_Sensor
- added MyoWare EMG Sensor2: ~, symbol MyoWare_EMG_Sensor:MyoWare_EMG_Sensor
- added MyoWare EMG Sensor3: ~, symbol MyoWare_EMG_Sensor:MyoWare_EMG_Sensor
- added MyoWare EMG Sensor4: ~, symbol MyoWare_EMG_Sensor:MyoWare_EMG_Sensor
- added U7: ADS1115IDGS, Package_SO:TSSOP-10_3x3mm_P0.5mm, symbol Analog_ADC:ADS1115IDGS
Connections:
- net +5V: now also M10.2 (+), M6.2 (+), M7.2 (+), M8.2 (+), M9.2 (+), MyoWare EMG Sensor1.1 (+Vs), MyoWare EMG Sensor2.1 (+Vs), MyoWare EMG Sensor3.1 (+Vs), MyoWare EMG Sensor4.1 (+Vs), U7.8 (VDD)
- net GND: now also M10.3 (-), M6.3 (-), M7.3 (-), M8.3 (-), M9.3 (-), MyoWare EMG Sensor1.2 (GND), MyoWare EMG Sensor2.2 (GND), MyoWare EMG Sensor3.2 (GND), MyoWare EMG Sensor4.2 (GND), U7.3 (GND)
- net at M2.1 (PWM): now also U1.P$4 (3V3/5V); no longer U1.P$14 (GPIO14)
- net at U1.P$11 (GPIO12): now also M6.1 (PWM)
- net at U1.P$7 (GPIO16): now also M7.1 (PWM)
- net at U1.P$6 (GPIO0): now also M8.1 (PWM)
- net at M1.1 (PWM): now also U1.P$2 (GPIO1); no longer U1.P$13 (GPIO15)
- net at U1.P$3 (GPIO3): now also M10.1 (PWM)
- net at U1.P$8 (3V3): now also M9.1 (PWM)
- new net: MyoWare EMG Sensor4.3 (SIG), U7.7 (AIN3)
- new net: MyoWare EMG Sensor2.3 (SIG), U7.5 (AIN1)
- new net: U1.P$14 (GPIO14), U7.1 (ADDR), U7.9 (SDA)
- new net: U1.P$13 (GPIO15), U7.10 (SCL)
- new net: MyoWare EMG Sensor1.3 (SIG), U7.4 (AIN0)
- new net: MyoWare EMG Sensor3.3 (SIG), U7.6 (AIN2)
- no-connect marks 6 -> 3
Other:
- moved on the sheet: C1
